File: docs/hardware/kicad/power_supply_v2/power_supply_v2.kicad_sch (KiCad schematic)
At the start: 118 parts, among them J1 Barrel_Jack, J2 LOAD 3V3, J3 LOAD 5V, J4 LOAD Vvar, M1 Fan_4pin, U1 TPS54302, U10 NUCLEO-G474RE, U11 INA180A3, U12 INA180A3, U13 INA180A1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

Commit message: fix missing pin assignment
Connections:
- net BTN_DSP_PC10: now reaches U10.CN7_1 (PC10)
- net BTN_DSP_PC10: now also S2.4 (B4)
- net BTN_V_{VAR}_PC11: now reaches U10.CN7_2 (PC11)
- net BTN_V_{VAR}_PC11: now also S2.3 (B3)
- net BTN_5VB_PC12: now reaches U10.CN7_3 (PC12)
- net BTN_5VB_PC12: now also S2.2 (B2)
- net RTRY_SW_PC1: now reaches U10.CN7_36 (PC1/PB9)
- net RTRY_SW_PC1: now also S1.4 (SW)
- net BTN_3V3B_PD2: now reaches U10.CN7_4 (PD2)
- net BTN_3V3B_PD2: now also S2.1 (B1)
- net OPAMP_3V3B_PB11: now reaches U10.CN10_18 (PB11)
- net OPAMP_3V3B_PB11: now also J2.1, R7.2
- net INA_5VB_OUT_PB2: now reaches U10.CN10_22 (PB2)
- net INA_5VB_OUT_PB2: now also C49.2, R30.2
- net BUCK_V_{VAR}_EN_PB15: now reaches U10.CN10_26 (PB15)
- net BUCK_V_{VAR}_EN_PB15: now also R22.1
- net BUCK_5V5_EN_PB13: now reaches U10.CN10_30 (PB13)
- net BUCK_5V5_EN_PB13: now also R8.2
- net BTN_3V3B_PB7: no longer names the net of U10.CN7_21 (PB7)
- net BTN_3V3B_PB7: no longer S2.1 (B1)
- net BTN_5VB_PC13: no longer names the net of U10.CN7_23 (PC13)
- net BTN_5VB_PC13: no longer S2.2 (B2)
- net BTN_DSP_PC15: no longer names the net of U10.CN7_27 (PC15)
- net BTN_DSP_PC15: no longer S2.4 (B4)
- net BTN_V_{VAR}_PC14: no longer names the net of U10.CN7_25 (PC14)
- net BTN_V_{VAR}_PC14: no longer S2.3 (B3)
- net BUCK_12V_EN_PC6: no longer names the net of U10.CN10_4 (PC6)
- net BUCK_12V_EN_PC6: no longer R18.1
- net BUCK_5V5_EN_PC8 renamed I2C3_SCL_PC8
- net I2C3_SCL_PC8: now also DS1.4 (SCL), DS2.4 (SCL), U14.4 (SCL), U15.4 (SCL); no longer R8.2
- net BUCK_V_{VAR}_EN_PC5 renamed LED_DATA_PC5
- net LED_DATA_PC5: now also U6.2 (1A); no longer R22.1
- net DAC_3V7_PA6 renamed DAC_3V3_PA6
- net DAC_5V5_PA5 renamed DAC_5V_PA5
- net FAN_PWM_PA12 renamed FAN_PWM_PB4
- net FAN_PWM_PB4: now also U10.CN10_27 (PB4); no longer U10.CN10_12 (PA12)
- net FAN_TACH_PA11 renamed FAN_TACH_PB10
- net FAN_TACH_PB10: now also U10.CN10_25 (PB10); no longer U10.CN10_14 (PA11)
- net HS_SW_3V3B_PC2 renamed HSSW_3V3B_PA12
- net HSSW_3V3B_PA12: now also U10.CN10_12 (PA12); no longer U10.CN7_35 (PC2)
- net HS_SW_5VB_PC3 renamed HSSW_5VB_PA11
- net HSSW_5VB_PA11: now also U10.CN10_14 (PA11); no longer U10.CN7_37 (PC3)
- removed net I2C1_SCL_PB8: DS1.4 (SCL), U10.CN10_3 (PB8), U14.4 (SCL)
- net I2C1_SDA_PB9 renamed I2C3_SDA_PC9
- net I2C3_SDA_PC9: now also DS2.3 (SDA), U10.CN10_1 (PC9), U15.1 (SDA); no longer U10.CN10_5 (PB9)
- removed net I2C2_SCL_PA9: DS2.4 (SCL), U10.CN10_21 (PA9), U15.4 (SCL)
- removed net I2C2_SDA_PA8: DS2.3 (SDA), U10.CN10_23 (PA8), U15.1 (SDA)
- net INA_20V_OUT_PB0 renamed INA_20V_OUT_PA9
- net INA_20V_OUT_PA9: now also U10.CN10_21 (PA9); no longer U10.CN7_34 (PB0)
- removed net INA_5VB_OUT_PB12: C49.2, R30.2, U10.CN10_16 (PB12)
- net INA_V_{VAR}_OUT_PB14 renamed INA_V_{VAR}_OUT_PA8
- net INA_V_{VAR}_OUT_PA8: now also U10.CN10_23 (PA8); no longer U10.CN10_28 (PB14)
- removed net LED_DATA_PC9: U10.CN10_1 (PC9), U6.2 (1A)
- net OPAMP_3V3A_PA1: no longer names the net of U10.CN7_30 (PA1)
- net OPAMP_3V3A_PA1: no longer R5.2
- removed net OPAMP_3V3B_PA7: J2.1, R7.2, U10.CN10_15 (PA7)
- net RTRY_CLK_PB5: no longer names the net of U10.CN10_29 (PB5)
- net RTRY_CLK_PB5: no longer S1.5 (CLK)
- net RTRY_DT_PB4 renamed RTRY_DT_PC2
- net RTRY_DT_PC2: now also U10.CN7_35 (PC2); no longer U10.CN10_27 (PB4)
- removed net RTRY_SW_PB10: S1.4 (SW), U10.CN10_25 (PB10)
- new net BUCK_12V_EN_PB14: R18.1, U10.CN10_28 (PB14)
- new net OPAMP_3V3A_PB12: R5.2, U10.CN10_16 (PB12)
- new net RTRY_CLK_PC3: S1.5 (CLK), U10.CN7_37 (PC3)
- no-connect marks 48 -> 55
